File: SteamDeck_Action_Buttons_Replacement_Pad.kicad_pcb (KiCad board)
At the start: 2 copper layers, 50.2 x 32.1 mm, 15 parts

Commit message: Updating with stiffener user.eco
Routing:
- net GND: track 25.3 -> 109.4 mm
